Commit message: Faithful LimX WF_TRON1A model + real tire grip
Make the model as realistic as the real LimX Dynamics robot:
- Pulled the actual limxdynamics/robot-description WF_TRON1A URDF and matched:
  * REAL inertials (full inertia tensors + COM) for base and all 8 leg links
    (total mass now 36.76 kg, real hip 2.3 kg, lower CoM 0.573 m above axle)
  * REAL mirrored joint axes (right leg hip/knee axes flipped) + asymmetric
    joint limits, exactly as the real robot
  * REAL actuator efforts: 80 N.m legs / 40 N.m wheels, 15/40 rad/s
  * joint damping, frictionloss, armature (rotor inertia); wheel friction 0.01
- Real tire grip: wheels now collide via a clean CYLINDER on the spin axis
  (friction mu=2.2) instead of the faceted convex-hull mesh -> rolls with
  traction, no slip. Mesh kept as visual only.
- Stance re-derived for the mirrored-axis convention (per-joint), balance
  re-tuned, gait re-tuned. URDF export also uses real inertials/efforts/axes.

Verified: balances, station-keeps, 120N shove, brief turns, 60s patrol upright,
gait (march/fwd/back/turn), RL env, both --check modes, regression all pass.

File: description/urdf/bravebot.urdf (robot description, URDF)
Before this commit: robot bravebot, 27 links, 26 joints
Links:
- link abadL_link: mass 1.4000 -> 1.4690
- link abadR_link: mass 1.4000 -> 1.4690
- link base_link: mass 9.0000 -> 9.5850
- link hipL_link: mass 1.6000 -> 2.3000
- link hipR_link: mass 1.6000 -> 2.3000
- link kneeL_link: mass 1.2000 -> 1.4900
- link kneeR_link: mass 1.2000 -> 1.4900
- link wheelL_link: mass 1.1000 -> 1.0800
- link wheelR_link: mass 1.1000 -> 1.0800
Joints:
- joint abad_L: limit lower=-0.5 upper=0.5 effort=60 velocity=15 -> lower=-0.38397 upper=1.39626 effort=80 velocity=15
- joint abad_R: limit lower=-0.5 upper=0.5 effort=60 velocity=15 -> lower=-1.39626 upper=0.38397 effort=80 velocity=15
- joint hip_L: limit lower=-1.2 upper=1.2 effort=60 velocity=15 -> lower=-1.01229 upper=1.39626 effort=80 velocity=15
- joint hip_R: axis 0 1 0 -> 0 -1 0; limit lower=-1.2 upper=1.2 effort=60 velocity=15 -> lower=-1.39626 upper=1.01229 effort=80 velocity=15
- joint knee_L: axis 0 1 0 -> 0 -1 0; limit lower=-2.2 upper=0.0 effort=60 velocity=15 -> lower=-0.87267 upper=1.36136 effort=80 velocity=15
- joint knee_R: limit lower=-2.2 upper=0.0 effort=60 velocity=15 -> lower=-1.36136 upper=0.87267 effort=80 velocity=15
- joint wheel_L: limit (none) -> effort=40 velocity=40
- joint wheel_R: limit (none) -> effort=40 velocity=40
